File: round-robin-10-72.kicad_sch (KiCad schematic)
At the start: 162 parts

Commit message: refactor: use dash-separated D{driving}-{driven} diode designators and fix 12-110 switch labels
Parts:
- renumbered D1 to D0-1, D2 to D0-2, D3 to D0-3, D4 to D0-4, D5 to D0-5, D6 to D0-6, D7 to D0-7, D8 to D0-8, D10 to D1-0, D12 to D1-2, D13 to D1-3, D14 to D1-4, D15 to D1-5, D16 to D1-6, D17 to D1-7, D18 to D1-8, D20 to D2-0, D21 to D2-1, D23 to D2-3, D24 to D2-4, D25 to D2-5, D26 to D2-6, D27 to D2-7, D28 to D2-8, D30 to D3-0, D31 to D3-1, D32 to D3-2, D34 to D3-4, D35 to D3-5, D36 to D3-6, D37 to D3-7, D38 to D3-8, D40 to D4-0, D41 to D4-1, D42 to D4-2, D43 to D4-3, D45 to D4-5, D46 to D4-6, D47 to D4-7, D48 to D4-8, D50 to D5-0, D51 to D5-1, D52 to D5-2, D53 to D5-3, D54 to D5-4, D56 to D5-6, D57 to D5-7, D58 to D5-8, D60 to D6-0, D61 to D6-1, D62 to D6-2, D63 to D6-3, D64 to D6-4, D65 to D6-5, D67 to D6-7, D68 to D6-8, D70 to D7-0, D71 to D7-1, D72 to D7-2, D73 to D7-3, D74 to D7-4, D75 to D7-5, D76 to D7-6, D78 to D7-8, D80 to D8-0, D81 to D8-1, D82 to D8-2, D83 to D8-3, D84 to D8-4, D85 to D8-5, D86 to D8-6, D87 to D8-7
