File: round-robin-12-110.kicad_sch (KiCad schematic)
At the start: 242 parts

Commit message: refactor: use dash-separated D{driving}-{driven} diode designators and fix 12-110 switch labels
Parts:
- renumbered D1 to D0-1, D110 to D0-10, D2 to D0-2, D3 to D0-3, D4 to D0-4, D5 to D0-5, D6 to D0-6, D7 to D0-7, D8 to D0-8, D9 to D0-9, D10 to D1-0, D111 to D1-10, D12 to D1-2, D13 to D1-3, D14 to D1-4, D15 to D1-5, D16 to D1-6, D17 to D1-7, D18 to D1-8, D19 to D1-9, D100 to D10-0, D101 to D10-1, D102 to D10-2, D103 to D10-3, D104 to D10-4, D105 to D10-5, D106 to D10-6, D107 to D10-7, D108 to D10-8, D109 to D10-9, D20 to D2-0, D21 to D2-1, D112 to D2-10, D23 to D2-3, D24 to D2-4, D25 to D2-5, D26 to D2-6, D27 to D2-7, D28 to D2-8, D29 to D2-9, D30 to D3-0, D31 to D3-1, D113 to D3-10, D32 to D3-2, D34 to D3-4, D35 to D3-5, D36 to D3-6, D37 to D3-7, D38 to D3-8, D39 to D3-9, D40 to D4-0, D41 to D4-1, D114 to D4-10, D42 to D4-2, D43 to D4-3, D45 to D4-5, D46 to D4-6, D47 to D4-7, D48 to D4-8, D49 to D4-9, D50 to D5-0, D51 to D5-1, D115 to D5-10, D52 to D5-2, D53 to D5-3, D54 to D5-4, D56 to D5-6, D57 to D5-7, D58 to D5-8, D59 to D5-9, D60 to D6-0, D61 to D6-1, D116 to D6-10, D62 to D6-2, D63 to D6-3, D64 to D6-4, D65 to D6-5, D67 to D6-7, D68 to D6-8, D69 to D6-9, D70 to D7-0, D71 to D7-1, D117 to D7-10, D72 to D7-2, D73 to D7-3, D74 to D7-4, D75 to D7-5, D76 to D7-6, D78 to D7-8, D79 to D7-9, D80 to D8-0, D81 to D8-1, D118 to D8-10, D82 to D8-2, D83 to D8-3, D84 to D8-4, D85 to D8-5, D86 to D8-6, D87 to D8-7, D89 to D8-9, D90 to D9-0, D91 to D9-1, D119 to D9-10, D92 to D9-2, D93 to D9-3, D94 to D9-4, D95 to D9-5, D96 to D9-6, D97 to D9-7, D98 to D9-8, RC1-1 to RC1-10, RC2-2 to RC2-10, RC3-3 to RC3-10, RC4-4 to RC4-10, RC5-5 to RC5-10, RC6-6 to RC6-10, RC7-7 to RC7-10, RC8-8 to RC8-10
