File: round-robin-7-30.kicad_sch (KiCad schematic)
At the start: 72 parts

Commit message: refactor: use dash-separated D{driving}-{driven} diode designators and fix 12-110 switch labels
Parts:
- renumbered D1 to D0-1, D2 to D0-2, D3 to D0-3, D4 to D0-4, D5 to D0-5, D10 to D1-0, D12 to D1-2, D13 to D1-3, D14 to D1-4, D15 to D1-5, D20 to D2-0, D21 to D2-1, D23 to D2-3, D24 to D2-4, D25 to D2-5, D30 to D3-0, D31 to D3-1, D32 to D3-2, D34 to D3-4, D35 to D3-5, D40 to D4-0, D41 to D4-1, D42 to D4-2, D43 to D4-3, D45 to D4-5, D50 to D5-0, D51 to D5-1, D52 to D5-2, D53 to D5-3, D54 to D5-4
Changed lines of the file:
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@@
 		(dnp no)
 		(fields_autoplaced yes)
-		(property "Reference" "D40"
+		(property "Reference" "D4-0"
 			(at 111.76 43.815 90)
 			(do_not_autoplace yes)
@@
 			(project "round-robin-7-30"
 				(path "/cbac505e-77a6-4a00-a758-435de33cca16"
-					(reference "D40")
+					(reference "D4-0")
 					(unit 1)
 				)
@@
 		(dnp no)
 		(fields_autoplaced yes)
-		(property "Reference" "D5"
+		(property "Reference" "D0-5"
 			(at 30.48 145.415 90)
 			(do_not_autoplace yes)
@@
 			(project "round-robin-7-30"
 				(path "/cbac505e-77a6-4a00-a758-435de33cca16"
-					(reference "D5")
+					(reference "D0-5")
 					(unit 1)
 				)
@@
 		(dnp no)
 		(fields_autoplaced yes)
-		(property "Reference" "D54"
+		(property "Reference" "D5-4"
 			(at 132.08 125.095 90)
 			(do_not_autoplace yes)
@@
 			(project "round-robin-7-30"
 				(path "/cbac505e-77a6-4a00-a758-435de33cca16"
-					(reference "D54")
+					(reference "D5-4")
 					(unit 1)
 				)
@@
 		(dnp no)
 		(fields_autoplaced yes)
-		(property "Reference" "D43"
+		(property "Reference" "D4-3"
 			(at 111.76 104.775 90)
 			(do_not_autoplace yes)
@@
 			(project "round-robin-7-30"
 				(path "/cbac505e-77a6-4a00-a758-435de33cca16"
-					(reference "D43")
+					(reference "D4-3")
 					(unit 1)
 				)
@@
 		(dnp no)
 		(fields_autoplaced yes)
-		(property "Reference" "D31"
+		(property "Reference" "D3-1"
 			(at 91.44 64.135 90)
 			(do_not_autoplace yes)
@@
 			(project "round-robin-7-30"
 				(path "/cbac505e-77a6-4a00-a758-435de33cca16"
-					(reference "D31")
+					(reference "D3-1")
 					(unit 1)
 				)
@@
 		(dnp no)
 		(fields_autoplaced yes)
-		(property "Reference" "D32"
+		(property "Reference" "D3-2"
 			(at 91.44 84.455 90)
 			(do_not_autoplace yes)
@@
 			(project "round-robin-7-30"
 				(path "/cbac505e-77a6-4a00-a758-435de33cca16"
-					(reference "D32")
+					(reference "D3-2")
 					(unit 1)
 				)
@@
 		(dnp no)
 		(fields_autoplaced yes)
-		(property "Reference" "D45"
+		(property "Reference" "D4-5"
 			(at 111.76 145.415 90)
 			(do_not_autoplace yes)
@@
 			(project "round-robin-7-30"
 				(path "/cbac505e-77a6-4a00-a758-435de33cca16"
-					(reference "D45")
+					(reference "D4-5")
 					(unit 1)
 				)
@@
 		(dnp no)
 		(fields_autoplaced yes)
-		(property "Reference" "D52"
+		(property "Reference" "D5-2"
 			(at 132.08 84.455 90)
 			(do_not_autoplace yes)
@@
 			(project "round-robin-7-30"
 				(path "/cbac505e-77a6-4a00-a758-435de33cca16"
-					(reference "D52")
+					(reference "D5-2")
 					(unit 1)
 				)
@@
 		(dnp no)
 		(fields_autoplaced yes)
-		(property "Reference" "D41"
+		(property "Reference" "D4-1"
 			(at 111.76 64.135 90)
 			(do_not_autoplace yes)
@@
 			(project "round-robin-7-30"
 				(path "/cbac505e-77a6-4a00-a758-435de33cca16"
-					(reference "D41")
+					(reference "D4-1")
 					(unit 1)
 				)
@@
 		(dnp no)
 		(fields_autoplaced yes)
-		(property "Reference" "D21"
+		(property "Reference" "D2-1"
 			(at 71.12 64.135 90)
 			(do_not_autoplace yes)
@@
 			(project "round-robin-7-30"
 				(path "/cbac505e-77a6-4a00-a758-435de33cca16"
-					(reference "D21")
+					(reference "D2-1")
 					(unit 1)
 				)
@@
 		(dnp no)
 		(fields_autoplaced yes)
-		(property "Reference" "D35"
+		(property "Reference" "D3-5"
 			(at 91.44 145.415 90)
 			(do_not_autoplace yes)
@@
 			(project "round-robin-7-30"
 				(path "/cbac505e-77a6-4a00-a758-435de33cca16"
-					(reference "D35")
+					(reference "D3-5")
 					(unit 1)
 				)
@@
 		(dnp no)
 		(fields_autoplaced yes)
-		(property "Reference" "D15"
+		(property "Reference" "D1-5"
 			(at 50.8 145.415 90)
 			(do_not_autoplace yes)
@@
 			(project "round-robin-7-30"
 				(path "/cbac505e-77a6-4a00-a758-435de33cca16"
-					(reference "D15")
+					(reference "D1-5")
 					(unit 1)
 				)
@@
 		(dnp no)
 		(fields_autoplaced yes)
-		(property "Reference" "D4"
+		(property "Reference" "D0-4"
 			(at 30.48 125.095 90)
 			(do_not_autoplace yes)
@@
 			(project "round-robin-7-30"
 				(path "/cbac505e-77a6-4a00-a758-435de33cca16"
-					(reference "D4")
+					(reference "D0-4")
 					(unit 1)
 				)
@@
 		(dnp no)
 		(fields_autoplaced yes)
-		(property "Reference" "D53"
+		(property "Reference" "D5-3"
 			(at 132.08 104.775 90)
 			(do_not_autoplace yes)
@@
 			(project "round-robin-7-30"
 				(path "/cbac505e-77a6-4a00-a758-435de33cca16"
-					(reference "D53")
+					(reference "D5-3")
 					(unit 1)
 				)
@@
 		(dnp no)
 		(fields_autoplaced yes)
-		(property "Reference" "D23"
+		(property "Reference" "D2-3"
 			(at 71.12 104.775 90)
 			(do_not_autoplace yes)
@@
 			(project "round-robin-7-30"
 				(path "/cbac505e-77a6-4a00-a758-435de33cca16"
-					(reference "D23")
+					(reference "D2-3")
 					(unit 1)
 				)
@@
 		(dnp no)
 		(fields_autoplaced yes)
-		(property "Reference" "D34"
+		(property "Reference" "D3-4"
 			(at 91.44 125.095 90)
 			(do_not_autoplace yes)
@@
 			(project "round-robin-7-30"
 				(path "/cbac505e-77a6-4a00-a758-435de33cca16"
-					(reference "D34")
+					(reference "D3-4")
 					(unit 1)
 				)
@@
 		(dnp no)
 		(fields_autoplaced yes)
-		(property "Reference" "D10"
+		(property "Reference" "D1-0"
 			(at 50.8 43.815 90)
 			(do_not_autoplace yes)
@@
 			(project "round-robin-7-30"
 				(path "/cbac505e-77a6-4a00-a758-435de33cca16"
-					(reference "D10")
+					(reference "D1-0")
 					(unit 1)
 				)
@@
 		(dnp no)
 		(fields_autoplaced yes)
-		(property "Reference" "D20"
+		(property "Reference" "D2-0"
 			(at 71.12 43.815 90)
 			(do_not_autoplace yes)
@@
 			(project "round-robin-7-30"
 				(path "/cbac505e-77a6-4a00-a758-435de33cca16"
-					(reference "D20")
+					(reference "D2-0")
 					(unit 1)
 				)
@@
 		(dnp no)
 		(fields_autoplaced yes)
-		(property "Reference" "D30"
+		(property "Reference" "D3-0"
 			(at 91.44 43.815 90)
 			(do_not_autoplace yes)
@@
 			(project "round-robin-7-30"
 				(path "/cbac505e-77a6-4a00-a758-435de33cca16"
-					(reference "D30")
+					(reference "D3-0")
 					(unit 1)
 				)
@@
 		(dnp no)
 		(fields_autoplaced yes)
-		(property "Reference" "D3"
+		(property "Reference" "D0-3"
 			(at 30.48 104.775 90)
 			(do_not_autoplace yes)
@@
 			(project "round-robin-7-30"
 				(path "/cbac505e-77a6-4a00-a758-435de33cca16"
-					(reference "D3")
+					(reference "D0-3")
 					(unit 1)
 				)
@@
 		(dnp no)
 		(fields_autoplaced yes)
-		(property "Reference" "D2"
+		(property "Reference" "D0-2"
 			(at 30.48 84.455 90)
 			(do_not_autoplace yes)
@@
 			(project "round-robin-7-30"
 				(path "/cbac505e-77a6-4a00-a758-435de33cca16"
-					(reference "D2")
+					(reference "D0-2")
 					(unit 1)
 				)
@@
 		(dnp no)
 		(fields_autoplaced yes)
-		(property "Reference" "D42"
+		(property "Reference" "D4-2"
 			(at 111.76 84.455 90)
 			(do_not_autoplace yes)
@@
 			(project "round-robin-7-30"
 				(path "/cbac505e-77a6-4a00-a758-435de33cca16"
-					(reference "D42")
+					(reference "D4-2")
 					(unit 1)
 				)
@@
 		(dnp no)
 		(fields_autoplaced yes)
-		(property "Reference" "D50"
+		(property "Reference" "D5-0"
 			(at 132.08 43.815 90)
 			(do_not_autoplace yes)
@@
 			(project "round-robin-7-30"
 				(path "/cbac505e-77a6-4a00-a758-435de33cca16"
-					(reference "D50")
+					(reference "D5-0")
 					(unit 1)
 				)
@@
 		(dnp no)
 		(fields_autoplaced yes)
-		(property "Reference" "D51"
+		(property "Reference" "D5-1"
 			(at 132.08 64.135 90)
 			(do_not_autoplace yes)
@@
 			(project "round-robin-7-30"
 				(path "/cbac505e-77a6-4a00-a758-435de33cca16"
-					(reference "D51")
+					(reference "D5-1")
 					(unit 1)
 				)
@@
 		(dnp no)
 		(fields_autoplaced yes)
-		(property "Reference" "D12"
+		(property "Reference" "D1-2"
 			(at 50.8 84.455 90)
 			(do_not_autoplace yes)
@@
 			(project "round-robin-7-30"
 				(path "/cbac505e-77a6-4a00-a758-435de33cca16"
-					(reference "D12")
+					(reference "D1-2")
 					(unit 1)
 				)
@@
 		(dnp no)
 		(fields_autoplaced yes)
-		(property "Reference" "D1"
+		(property "Reference" "D0-1"
 			(at 30.48 64.135 90)
 			(do_not_autoplace yes)
@@
 			(project "round-robin-7-30"
 				(path "/cbac505e-77a6-4a00-a758-435de33cca16"
-					(reference "D1")
+					(reference "D0-1")
 					(unit 1)
 				)
@@
 		(dnp no)
 		(fields_autoplaced yes)
-		(property "Reference" "D14"
+		(property "Reference" "D1-4"
 			(at 50.8 125.095 90)
 			(do_not_autoplace yes)
@@
 			(project "round-robin-7-30"
 				(path "/cbac505e-77a6-4a00-a758-435de33cca16"
-					(reference "D14")
+					(reference "D1-4")
 					(unit 1)
 				)
@@
 		(dnp no)
 		(fields_autoplaced yes)
-		(property "Reference" "D24"
+		(property "Reference" "D2-4"
 			(at 71.12 125.095 90)
 			(do_not_autoplace yes)
@@
 			(project "round-robin-7-30"
 				(path "/cbac505e-77a6-4a00-a758-435de33cca16"
-					(reference "D24")
+					(reference "D2-4")
 					(unit 1)
 				)
@@
 		(dnp no)
 		(fields_autoplaced yes)
-		(property "Reference" "D13"
+		(property "Reference" "D1-3"
 			(at 50.8 104.775 90)
 			(do_not_autoplace yes)
@@
 			(project "round-robin-7-30"
 				(path "/cbac505e-77a6-4a00-a758-435de33cca16"
-					(reference "D13")
+					(reference "D1-3")
 					(unit 1)
 				)
@@
 		(dnp no)
 		(fields_autoplaced yes)
-		(property "Reference" "D25"
+		(property "Reference" "D2-5"
 			(at 71.12 145.415 90)
 			(do_not_autoplace yes)
@@
 			(project "round-robin-7-30"
 				(path "/cbac505e-77a6-4a00-a758-435de33cca16"
-					(reference "D25")
+					(reference "D2-5")
 					(unit 1)
 				)
